Commit message: more work done on hip  control -- not functional yet!

File: hip_assembly/urdf/hip_assembly.urdf (robot description, URDF)
Before this commit: robot hip_assembly, 2 links, 1 joints
Joints:
- removed joint Joint_1
- added joint hip_revolute_joint: type revolute, parent Link_1, child Link_2, origin xyz=-0.12828 0.11233 0.10668 rpy=1.542 1.2658 -0.030421, axis 0 0 1, limit lower=0 upper=3.14 effort=50 velocity=4

Commit message: brought ros_control to a functional state

File: hip_assembly/urdf/hip_assembly.urdf (robot description, URDF)
Before this commit: robot hip_assembly, 2 links, 1 joints
Joints:
- joint hip_revolute_joint: limit lower=0 upper=3.14 effort=50 velocity=4 -> lower=0 upper=2.2 effort=10 velocity=0.5
